Commit message: fixed torso pitch to 10deg

File: urdf/ergoCub/robots/ergoCubSN001/model.urdf (robot description, URDF)
Before this commit: robot ergoCub, 204 links, 203 joints
Joints:
- joint torso_pitch: limit lower=-0.3141592653589793 upper=0.7853981633974483 effort=1e+9 velocity=1e+9 -> (none); origin xyz=-7.30886630439206e-17 -4.930380657631324e-32 0.11800000000000001 rpy=3.9719461100401744e-15 2.710505431213761e-20 1.0587911275090697e-22 -> xyz=-7.30886630439206e-17 -4.930380657631324e-32 0.11800000000000001 rpy=3.9719461100401744e-15 0.174533 1.0587911275090697e-22; type revolute -> fixed

Commit message: Revert "fixed torso pitch to 10deg"
This reverts commit 1d63ae7228943c863d387b447b21bdf59f451518.

File: urdf/ergoCub/robots/ergoCubSN001/model.urdf (robot description, URDF)
Before this commit: robot ergoCub, 204 links, 203 joints
Joints:
- joint torso_pitch: limit (none) -> lower=-0.3141592653589793 upper=0.7853981633974483 effort=1e+9 velocity=1e+9; origin xyz=-7.30886630439206e-17 -4.930380657631324e-32 0.11800000000000001 rpy=3.9719461100401744e-15 0.174533 1.0587911275090697e-22 -> xyz=-7.30886630439206e-17 -4.930380657631324e-32 0.11800000000000001 rpy=3.9719461100401744e-15 2.710505431213761e-20 1.0587911275090697e-22; type fixed -> revolute
