Commit message: first commit for stereo cameras on 1_1

File: urdf/ergoCub/robots/ergoCubGazeboV1_1/model.urdf (robot description, URDF)
Before this commit: robot ergoCub, 204 links, 203 joints
Links:
- added link left_stereo_frame
- added link right_stereo_frame
Joints:
- added joint left_stereo_frame_frame_fixed_joint: type fixed, parent realsense_rgb_frame, child left_stereo_frame, origin xyz=-0.59 0.0 0.0 rpy=0.0 0.0 0.0
- added joint right_stereo_frame_fixed_joint: type fixed, parent realsense_rgb_frame, child right_stereo_frame, origin xyz=0.36 0.0 0.0 rpy=0.0 0.0 0.0

Commit message: not working: stereo cam

File: urdf/ergoCub/robots/ergoCubGazeboV1_1/model.urdf (robot description, URDF)
Before this commit: robot ergoCub, 206 links, 205 joints
Joints:
- joint left_stereo_frame_frame_fixed_joint: origin xyz=-0.59 0.0 0.0 rpy=0.0 0.0 0.0 -> xyz=-0.059 0.0 0.0 rpy=0.0 0.0 0.0
- joint right_stereo_frame_fixed_joint: origin xyz=0.36 0.0 0.0 rpy=0.0 0.0 0.0 -> xyz=0.036 0.0 0.0 rpy=0.0 0.0 0.0
